File: Project/Electronics/FluidNC-ESP32-XIAO/FluidNC-ESP32-XIAO.kicad_pcb (KiCad board)
At the start: 2 copper layers, 24 parts, among them J1 Tirette, J2 Team, J3 BAU, J4 OledI2C, J5 Conn_01x04, J6 Conn_01x04, J7 SensorUltrasonic, J8 ConBatt, M1 Motor_Servo, SW1 SW_DIP_x02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

Commit message: Create Board - WIP
Parts:
- removed D2: LED_Small, LED_SMD:LED_1206_3216Metric_Pad1.42x1.75mm_HandSolder
- removed J3: BAU, Connector_Molex:Molex_KK-254_AE-6410-02A_1x02_P2.54mm_Vertical
- added C3: 10uF 25V, Capacitor_THT:C_Disc_D6.0mm_W2.5mm_P5.00mm, F.Cu at (144.0, 116.0)
- added C4: 10uF 25V, Capacitor_THT:C_Disc_D6.0mm_W2.5mm_P5.00mm, F.Cu at (157.0, 116.0)
- added D3: 5mm Red, LED_THT:LED_D5.0mm, F.Cu at (161.5, 111.0)
- added R3: 4,7K, Resistor_THT:R_Axial_DIN0204_L3.6mm_D1.6mm_P7.62mm_Horizontal, F.Cu at (146.1, 70.6)
- added R5: 1K, Resistor_THT:R_Axial_DIN0204_L3.6mm_D1.6mm_P7.62mm_Horizontal, F.Cu at (166.6, 116.1)
- added SW6: CherryMX, Button_Switch_Keyboard:SW_Cherry_MX_1.00u_PCB, F.Cu at (160.3, 67.6)
- added U5: R-78E5.0-1.0, Converter_DCDC:Converter_DCDC_RECOM_R-78E-0.5_THT, F.Cu at (147.9, 111.2)
- D1: value D_Schottky -> 1N5819
- J1: value Tirette -> Limit_X
- J2: value Team -> Limit_Y
- J7: value SensorUltrasonic -> BAU; footprint Connector_PinHeader_2.54mm:PinHeader_1x04_P2.54mm_Vertical -> Connector_Molex:Molex_KK-254_AE-6410-02A_1x02_P2.54mm_Vertical
- J8: value ConBatt -> Barrel_Jack_Switch; footprint Connector_Molex:Molex_KK-396_A-41791-0002_1x02_P3.96mm_Vertical -> Connector_BarrelJack:BarrelJack_Horizontal
- R1: footprint Resistor_SMD:R_1206_3216Metric_Pad1.30x1.75mm_HandSolder -> Resistor_THT:R_Axial_DIN0204_L3.6mm_D1.6mm_P7.62mm_Horizontal
- R2: value 1K -> 4,7K; footprint Resistor_SMD:R_1206_3216Metric_Pad1.30x1.75mm_HandSolder -> Resistor_THT:R_Axial_DIN0204_L3.6mm_D1.6mm_P7.62mm_Horizontal
- moved H3 95.5 mm to (119.0, 136.0)
- moved H1 88.2 mm to (119.0, 69.0)
- moved C1 62.4 mm to (120.9, 108.2), turned to 90 degrees
- moved R2 61.0 mm to (146.1, 73.2), turned to 180 degrees
- moved C2 59.9 mm to (131.1, 134.7)
- moved R1 58.0 mm to (145.0, 78.0), turned to 180 degrees
- moved SW2 49.4 mm to (150.9, 124.9), turned to 180 degrees
- moved H4 46.8 mm to (171.0, 136.0)
- moved SW1 41.7 mm to (150.9, 99.5), turned to 180 degrees
- moved H2 40.8 mm to (171.0, 69.0)
- moved J4 40.6 mm to (146.1, 67.3), turned to -90 degrees
- moved U3 37.8 mm to (133.7, 118.6)
- moved M1 34.8 mm to (133.9, 78.0), turned to -90 degrees
- moved J7 27.6 mm to (151.5, 134.0)
- moved J1 27.1 mm to (121.6, 76.0), turned to -90 degrees
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Connections:
- C1 pad 1: +5V -> +12V
- C2 pad 1: +5V -> +12V
- J7 pad 1: SDA -> +12V
- J7 pad 2: SCL -> +BATT
- R2 pad 1: +5V -> SCL
- R2 pad 2: Net-(D2-A) -> +3.3V
- U1 pad 1: EN -> Key01
- U1 pad 10: switch_2 -> DirY
- U1 pad 11: unconnected-(U1-GPIO9/D10/A10/MOSI-Pad11) -> StepY
- U1 pad 2: StepG -> Servo
- U1 pad 3: DirG -> switch_1
- U1 pad 4: StepD -> switch_2
- U1 pad 7: DirD -> DirX
- U1 pad 8: Servo -> StepX
- U1 pad 9: switch_1 -> EN
- U2 pad 10: StepG -> StepX
- U2 pad 3: Net-(J5-Pin_3) -> Net-(J5-Pin_1)
- U2 pad 4: Net-(J5-Pin_1) -> Net-(J5-Pin_2)
- U2 pad 5: Net-(J5-Pin_2) -> Net-(J5-Pin_3)
- U2 pad 8: +5V -> +12V
- U2 pad 9: DirG -> DirX
- U3 pad 10: StepD -> StepY
- U3 pad 3: Net-(J6-Pin_3) -> Net-(J6-Pin_1)
- U3 pad 4: Net-(J6-Pin_1) -> Net-(J6-Pin_2)
- U3 pad 5: Net-(J6-Pin_2) -> Net-(J6-Pin_3)
- U3 pad 8: +5V -> +12V
- U3 pad 9: DirD -> DirY
Routing:
- net +3.3V: track 0.00 -> 137.3 mm, vias 0 -> 1
- net +12V: track 0.00 -> 101.3 mm
- net +5V: track 0.00 -> 74.5 mm, vias 0 -> 2
- net switch_1: track 0.00 -> 50.6 mm
- net EN: track 0.00 -> 49.5 mm
- net switch_2: track 0.00 -> 44.5 mm
- net StepY: track 0.00 -> 29.4 mm
- net Servo: track 0.00 -> 27.3 mm
- net StepX: track 0.00 -> 27.2 mm
- net DirY: track 0.00 -> 26.3 mm
- net SCL: track 0.00 -> 25.7 mm
- net SDA: track 0.00 -> 24.5 mm
- net Key01: track 0.00 -> 23.0 mm
- net DirX: track 0.00 -> 17.6 mm
- net +BATT: track 0.00 -> 13.3 mm
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- added copper zone on B.Cu, net GND
- added copper zone on F.Cu, net GND
Other:
- board outline added: 60 x 75 mm
