File: Project/Electronics/FluidNC-ESP32-XIAO/FluidNC-ESP32-XIAO.kicad_sch (KiCad schematic)
At the start: 23 parts, among them J1 Tirette, J2 Team, J3 BAU, J4 OledI2C, J5 Conn_01x04, J6 Conn_01x04, J8 ConBatt, M1 Motor_Servo, SW1 SW_DIP_x02, SW2 SW_DIP_x02, U1 XIAO-ESP32-S3-DIP, U2 TMC2209_SILENTSTEPSTICK, U3 TMC2209_SILENTSTEPSTICK

Commit message: Create Board - WIP
Parts:
- removed D2: LED_Small, LED_SMD:LED_1206_3216Metric_Pad1.42x1.75mm_HandSolder, symbol Device:LED_Small
- removed J3: BAU, Connector_Molex:Molex_KK-254_AE-6410-02A_1x02_P2.54mm_Vertical, symbol Connector_Generic:Conn_01x02
- removed J8: ConBatt, Connector_Molex:Molex_KK-396_A-41791-0002_1x02_P3.96mm_Vertical, symbol Connector_Generic:Conn_01x02
- removed R2: 1K, Resistor_SMD:R_1206_3216Metric_Pad1.30x1.75mm_HandSolder, symbol Device:R_Small
- added C3, C4: 10uF 25V, Capacitor_THT:C_Disc_D6.0mm_W2.5mm_P5.00mm, symbol Device:C_Small
- added D3: 5mm Red, LED_THT:LED_D5.0mm, symbol Device:LED_Small
- added J3: Conn_02x08_Odd_Even, Connector_PinHeader_2.54mm:PinHeader_2x08_P2.54mm_Vertical, symbol Connector_Generic:Conn_02x08_Odd_Even
- added J7: BAU, Connector_Molex:Molex_KK-254_AE-6410-02A_1x02_P2.54mm_Vertical, symbol Connector_Generic:Conn_01x02
- added J8: Barrel_Jack_Switch, Connector_BarrelJack:BarrelJack_Horizontal, symbol Connector:Barrel_Jack_Switch
- added R3, R4: 4.7K, Resistor_THT:R_Axial_DIN0204_L3.6mm_D1.6mm_P7.62mm_Horizontal, symbol Device:R_Small
- added R5: 1K, Resistor_THT:R_Axial_DIN0204_L3.6mm_D1.6mm_P7.62mm_Horizontal, symbol Device:R_Small
- added U4: PCF8574P, Package_DIP:DIP-16_W7.62mm, symbol Interface_Expansion:PCF8574P
- added U5: R-78E5.0-1.0, Converter_DCDC:Converter_DCDC_RECOM_R-78E-0.5_THT, symbol Regulator_Switching:R-78E5.0-1.0
- D1: value D_Schottky -> 1N5819
- J1: value Tirette -> Limit_X
- J2: value Team -> Limit_Y
- R1: footprint Resistor_SMD:R_1206_3216Metric_Pad1.30x1.75mm_HandSolder -> Resistor_THT:R_Axial_DIN0204_L3.6mm_D1.6mm_P7.62mm_Horizontal
Connections:
- net +3.3V: now also R3.2, R4.2, U4.16 (VDD)
- net +5V: now also C4.1, R5.1, U5.3 (OUT); no longer C1.1, C2.1, U2.8 (VM), U3.8 (VM)
- net +BATT: now also J7.2 (Pin_2), J8.1
- net EN: now also U1.9 (GPIO7/D8/A8/SCK); no longer U1.1 (GPIO1/D0/A0)
- net GND: now also C3.2, C4.2, D3.1 (K), J3.1 (Pin_1), J3.11 (Pin_11), J3.13 (Pin_13), J3.15 (Pin_15), J3.3 (Pin_3), J3.5 (Pin_5), J3.7 (Pin_7), J3.9 (Pin_9), J8.2, J8.3, U4.1 (A0), U4.2 (A1), U4.3 (A2), U4.8 (GND), U5.2 (GND)
- net SCL: now also R3.1, U4.14 (SCL)
- net SDA: now also R4.1, U4.15 (SDA)
- net Servo: now also U1.2 (GPIO2/DA/A1); no longer U1.8 (U0RXD/D7/RX)
- net switch_1: now also U1.3 (GPIO3/D2/A2); no longer U1.9 (GPIO7/D8/A8/SCK)
- net switch_2: now also U1.4 (GPIO4/D3/A3); no longer U1.10 (GPIO8/D9/A9/MISO)
- net at J6.1 (Pin_1): now also U3.3 (M1B); no longer U3.4 (M1A)
- net at J6.2 (Pin_2): now also U3.4 (M1A); no longer U3.5 (M2A)
- net at J6.3 (Pin_3): now also U3.5 (M2A); no longer U3.3 (M1B)
- net at U2.3 (M1B): now also J5.1 (Pin_1); no longer J5.3 (Pin_3)
- net at U2.4 (M1A): now also J5.2 (Pin_2); no longer J5.1 (Pin_1)
- net at U2.5 (M2A): now also J5.3 (Pin_3); no longer J5.2 (Pin_2)
- net StepY: now reaches U1.11 (GPIO9/D10/A10/MOSI)
- net StepY: now also U3.10 (STEP)
- net DirD renamed DirX
- net DirX: now also U2.9 (DIR); no longer U3.9 (DIR)
- removed net DirG: U1.3 (GPIO3/D2/A2), U2.9 (DIR)
- removed net StepD: U1.4 (GPIO4/D3/A3), U3.10 (STEP)
- net StepG renamed StepX
- net StepX: now also U1.8 (U0RXD/D7/RX); no longer U1.2 (GPIO2/DA/A1)
- new net: J3.12 (Pin_12), U4.10 (P5)
- new net: J3.14 (Pin_14), U4.11 (P6)
- new net: J3.16 (Pin_16), U4.12 (P7)
- new net: J3.2 (Pin_2), U4.4 (P0)
- new net: J3.4 (Pin_4), U4.5 (P1)
- new net: J3.6 (Pin_6), U4.6 (P2)
- new net: J3.8 (Pin_8), U4.7 (P3)
- new net: J3.10 (Pin_10), U4.9 (P4)
- new net: D3.2 (A), R5.2
- new net +12V: C1.1, C2.1, C3.1, J7.1 (Pin_1), U2.8 (VM), U3.8 (VM), U5.1 (IN)
- new net DirY: U1.10 (GPIO8/D9/A9/MISO), U3.9 (DIR)
Other:
- moved on the sheet: C1, C2, D1, J1, J2, J4, J5, J6, M1, R1, SW1, U1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

Commit message: new cnc shield MKS
Parts:
- removed J3: Conn_02x08_Odd_Even, Connector_PinHeader_2.54mm:PinHeader_2x08_P2.54mm_Vertical, symbol Connector_Generic:Conn_02x08_Odd_Even
- removed R4: 4.7K, Resistor_THT:R_Axial_DIN0204_L3.6mm_D1.6mm_P7.62mm_Horizontal, symbol Device:R_Small
- removed U4: PCF8574P, Package_DIP:DIP-16_W7.62mm, symbol Interface_Expansion:PCF8574P
- added R2: 4,7K, Resistor_THT:R_Axial_DIN0204_L3.6mm_D1.6mm_P7.62mm_Horizontal, symbol Device:R_Small
- added SW6: CherryMX, Button_Switch_Keyboard:SW_Cherry_MX_1.00u_PCB, symbol Switch:SW_Push
- R3: value 4.7K -> 4,7K
Connections:
- net +3.3V: now also R2.2
- net GND: now also SW6.2
- net SCL: now also R2.1; no longer R3.1
- net SDA: now also R3.1
- net Key01: now reaches U1.1 (GPIO1/D0/A0)
- net Key01: now also SW6.1
