File: Project/Electronics/CNC-Shield-MKS/CNC-Shield-MKS.kicad_pcb (KiCad board)
At the start: 2 copper layers, 68.6 x 53.3 mm, 20 parts, among them J1 Power, J10 Microstepping, J11 Microstepping, J12 Y_Stepper, J2 Digital/PWM, J3 Analog, J4 Digital/PWM, J5 Servomoteur, J6 X-Limit-Switch, J7 Y-Limit-Switch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

Commit message: new CNC shield MKS
Parts:
- added C1: 100uF, Capacitor_THT:CP_Radial_D8.0mm_P3.50mm, F.Cu at (164.8, 77.6)
- added C2: 100uF, Capacitor_THT:CP_Radial_D8.0mm_P3.50mm, F.Cu at (143.3, 77.7)
- added C3: 10uF 25V, Capacitor_THT:C_Disc_D6.0mm_W2.5mm_P5.00mm, F.Cu at (109.5, 67.8)
- added C4: 10uF 25V, Capacitor_THT:C_Disc_D6.0mm_W2.5mm_P5.00mm, F.Cu at (110.7, 52.5)
- added D2: 5mm Green, LED_THT:LED_D5.0mm, F.Cu at (102.9, 50.8)
- added G***: LOGO, LOGO, F.Cu at (143.3, 88.6)
- added G***: LOGO, LOGO, F.Cu at (143.7, 71.6)
- added G***: LOGO, LOGO, F.Cu at (163.6, 93.5)
- added G***: LOGO, LOGO, F.Cu at (119.5, 71.6)
- added G***: LOGO, LOGO, F.Cu at (117.3, 91.2)
- added G***: LOGO, LOGO, F.Cu at (110.2, 98.6)
- added G***: LOGO, LOGO, F.Cu at (128.0, 88.6)
- added J13: HID, Connector_PinHeader_2.54mm:PinHeader_2x03_P2.54mm_Vertical, F.Cu at (161.0, 86.1)
- added R2: 1K, Resistor_THT:R_Axial_DIN0204_L3.6mm_D1.6mm_P5.08mm_Horizontal, F.Cu at (113.7, 49.5)
- added R3: 220, Resistor_THT:R_Axial_DIN0204_L3.6mm_D1.6mm_P5.08mm_Horizontal, F.Cu at (119.9, 78.0)
- added U2: R-78E5.0-1.0, Converter_DCDC:Converter_DCDC_RECOM_R-78E-0.5_THT, F.Cu at (113.2, 62.7)
- added kibuzzard-68AC6E26: G***, kibuzzard-68AC6E26, F.Cu at (128.5, 93.5)
- added kibuzzard-68AC6E2C: G***, kibuzzard-68AC6E2C, F.Cu at (143.8, 93.5)
- added kibuzzard-68AC6E46: G***, kibuzzard-68AC6E46, F.Cu at (151.3, 93.4)
- added kibuzzard-68AC6E4C: G***, kibuzzard-68AC6E4C, F.Cu at (136.1, 93.4)
- added kibuzzard-68AC6EBA: G***, kibuzzard-68AC6EBA, F.Cu at (121.2, 93.4)
- added kibuzzard-68AC6EE0: G***, kibuzzard-68AC6EE0, F.Cu at (122.9, 88.7)
- added kibuzzard-68AC6EF6: G***, kibuzzard-68AC6EF6, F.Cu at (127.6, 91.2)
- added kibuzzard-68AC6EF6: G***, kibuzzard-68AC6EF6, F.Cu at (142.8, 91.2)
- added kibuzzard-68AC6F25: G***, kibuzzard-68AC6F25, F.Cu at (123.0, 86.1)
- added kibuzzard-68AC6F3F: G***, kibuzzard-68AC6F3F, F.Cu at (143.0, 86.1)
- added kibuzzard-68AC6F3F: G***, kibuzzard-68AC6F3F, F.Cu at (127.8, 86.1)
- added kibuzzard-68AC6F70: G***, kibuzzard-68AC6F70, F.Cu at (156.8, 86.1)
- added kibuzzard-68AC6F8C: G***, kibuzzard-68AC6F8C, F.Cu at (157.2, 88.6)
- added kibuzzard-68AC6F9A: G***, kibuzzard-68AC6F9A, F.Cu at (156.7, 91.2)
- added kibuzzard-68AC6FF4: G***, kibuzzard-68AC6FF4, F.Cu at (124.9, 73.9)
- added kibuzzard-68AC7005: G***, kibuzzard-68AC7005, F.Cu at (149.0, 73.9)
- added kibuzzard-68AC7035: G***, kibuzzard-68AC7035, F.Cu at (137.2, 68.3)
- added kibuzzard-68AC7035: G***, kibuzzard-68AC7035, F.Cu at (161.3, 68.3)
- added kibuzzard-68AC7044: G***, kibuzzard-68AC7044, F.Cu at (134.6, 68.3)
- added kibuzzard-68AC7044: G***, kibuzzard-68AC7044, F.Cu at (158.8, 68.3)
- added kibuzzard-68AC7048: G***, kibuzzard-68AC7048, F.Cu at (132.1, 68.3)
- added kibuzzard-68AC7048: G***, kibuzzard-68AC7048, F.Cu at (156.2, 68.3)
- added kibuzzard-68AC7082: G***, kibuzzard-68AC7082, F.Cu at (102.9, 62.0)
- added kibuzzard-68AC71B3: G***, kibuzzard-68AC71B3, F.Cu at (116.6, 79.2)
- D1: value RED -> 5mm RED
- J1, J4: footprint Connector_PinSocket_2.54mm:PinSocket_1x08_P2.54mm_Vertical -> Connector_PinHeader_2.54mm:PinHeader_1x08_P2.54mm_Vertical; moved to B.Cu
- J2: footprint Connector_PinSocket_2.54mm:PinSocket_1x10_P2.54mm_Vertical -> Connector_PinHeader_2.54mm:PinHeader_1x10_P2.54mm_Vertical; moved to B.Cu
- J3: footprint Connector_PinSocket_2.54mm:PinSocket_1x06_P2.54mm_Vertical -> Connector_PinHeader_2.54mm:PinHeader_1x06_P2.54mm_Vertical; moved to B.Cu
- moved J5 39.2 mm to (119.9, 86.1), turned to 0 degrees
- moved J7 27.5 mm to (130.6, 86.1), turned to 0 degrees
- moved J9 23.5 mm to (149.4, 83.6), turned to 0 degrees
- moved J6 23.2 mm to (145.8, 86.1), turned to 0 degrees
- moved J12 20.4 mm to (134.1, 83.6), turned to 0 degrees
- moved A2 19.5 mm to (121.9, 71.5)
- moved J11 19.4 mm to (132.1, 65.0)
- moved JP1 18.8 mm to (151.1, 62.3), turned to -90 degrees
- moved JP2 18.7 mm to (127.0, 62.3), turned to -90 degrees
- moved J10 17.2 mm to (156.2, 65.0)
- moved A1 17.1 mm to (146.1, 71.5)
- moved F1 12.5 mm to (110.5, 84.1), turned to 90 degrees
- moved J8 8.54 mm to (110.2, 93.0), turned to 0 degrees
- moved D1 1.21 mm to (102.9, 84.8)
- moved SW2 0.54 mm to (102.6, 71.4)
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Connections:
- J2 pad 1: /SCL/A5 -> /SCL
- J2 pad 2: /SDA/A4 -> /SDA
- J3 pad 1: /A0 -> Reset/Abord
- J3 pad 2: /A1 -> Feed/Hold
- J3 pad 3: /A2 -> Start/Resume
- J5 pad 1: Servo -> Net-(J5-Pin_1)
- J5 pad 2: +5V -> +5P
Routing:
- net +5V: track 0.00 -> 106.2 mm
- net +12V: track 0.00 -> 106.2 mm
- net Y_Limit: track 0.00 -> 61.5 mm
- net +5P: track 0.00 -> 48.5 mm
- net X_Limit: track 0.00 -> 44.6 mm
- net Servo: track 0.00 -> 43.5 mm
- net EnMotors: track 0.00 -> 38.2 mm
- net Y_STEP: track 0.00 -> 38.0 mm
- net Y_DIR: track 0.00 -> 33.3 mm
- net Net-(A2-2B): track 0.00 -> 24.4 mm
- net Net-(A1-2B): track 0.00 -> 24.3 mm
- net Net-(A2-2A): track 0.00 -> 21.1 mm
- net Net-(A1-2A): track 0.00 -> 21.0 mm
- net Net-(A2-1A): track 0.00 -> 18.7 mm
- net Net-(A1-1A): track 0.00 -> 18.2 mm
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- added copper zone on B.Cu, net GND
- added copper zone on F.Cu, net GND
