File: Project/Electronics/CNC-Shield-MKS/CNC-Shield-MKS.kicad_sch (KiCad schematic)
At the start: 22 parts, among them J1 Power, J10 Microstepping, J11 Microstepping, J12 Y_Stepper, J2 Digital/PWM, J3 Analog, J4 Digital/PWM, J5 Servomoteur, J6 X-Limit-Switch, J7 Y-Limit-Switch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

Commit message: new CNC shield MKS
Parts:
- added C3, C4: 10uF 25V, Capacitor_THT:C_Disc_D6.0mm_W2.5mm_P5.00mm, symbol Device:C_Small
- added D2: 5mm Green, LED_THT:LED_D5.0mm, symbol Device:LED_Small
- added J13: Microstepping, Connector_PinHeader_2.54mm:PinHeader_2x03_P2.54mm_Vertical, symbol Connector_Generic:Conn_02x03_Odd_Even
- added R2: 1K, Resistor_THT:R_Axial_DIN0204_L3.6mm_D1.6mm_P5.08mm_Horizontal, symbol Device:R_Small
- added R3: 220, Resistor_THT:R_Axial_DIN0204_L3.6mm_D1.6mm_P5.08mm_Horizontal, symbol Device:R_Small
- added U2: R-78E5.0-1.0, Converter_DCDC:Converter_DCDC_RECOM_R-78E-0.5_THT, symbol Regulator_Switching:R-78E5.0-1.0
- C1, C2: footprint (none) -> Capacitor_THT:CP_Radial_D8.0mm_P3.50mm; Gotronic (none) -> 22711
- D1: value RED -> 5mm RED
- J1, J4: footprint Connector_PinSocket_2.54mm:PinSocket_1x08_P2.54mm_Vertical -> Connector_PinHeader_2.54mm:PinHeader_1x08_P2.54mm_Vertical
- J2: footprint Connector_PinSocket_2.54mm:PinSocket_1x10_P2.54mm_Vertical -> Connector_PinHeader_2.54mm:PinHeader_1x10_P2.54mm_Vertical
- J3: footprint Connector_PinSocket_2.54mm:PinSocket_1x06_P2.54mm_Vertical -> Connector_PinHeader_2.54mm:PinHeader_1x06_P2.54mm_Vertical
Connections:
- net +12V: now also C3.1, U2.1 (IN)
- net +5V: no longer J5.2 (Pin_2)
- net GND: now also C3.2, C4.2, D2.1 (K), J13.2 (Pin_2), J13.4 (Pin_4), J13.6 (Pin_6), U2.2 (GND)
- net SCL/A5: no longer J2.1 (Pin_1)
- net SDA/A4: no longer J2.2 (Pin_2)
- net Servo: now also R3.1; no longer J5.1 (Pin_1)
- net A0 renamed Reset/Abord
- net Reset/Abord: now also J13.1 (Pin_1)
- net A1 renamed Feed/Hold
- net Feed/Hold: now also J13.3 (Pin_3)
- net A2 renamed Start/Resume
- net Start/Resume: now also J13.5 (Pin_5)
- new net: D2.2 (A), R2.2
- new net: J5.1 (Pin_1), R3.2
- new net +5P: C4.1, J5.2 (Pin_2), R2.1, U2.3 (OUT)
- new net SCL: J2.1 (Pin_1)
- new net SDA: J2.2 (Pin_2)
Other:
- moved on the sheet: C1, D1, F1, J5, J6, J7, J8, R1, SW2
